File: esp8266-board/esp8266-board.sch (KiCad schematic (older format))
At the start: 25 parts, among them J1 PGM, J2 StepDown-3A, J3 LED, J4 USB, J5 Barrel_Jack, U1 ESP-12E, U2 AP2112, U3 AMS1117-3.3

Commit message: First board rev order 0.1
Parts:
- C5: renamed from C?; footprint (none) -> Capacitors_THT:CP_Radial_D8.0mm_P5.00mm
Connections:
- net GND: now also J5.3
- no-connect marks 17 -> 16
Changed lines of the file:
@@
 NoConn ~ 4650 3600
 NoConn ~ 4550 3600
-NoConn ~ 9750 1550
 Text GLabel 1950 2400 0    60   Input ~ 0
 ADC
@@
 $EndComp
 $Comp
-L CP C?
+L CP C5
 U 1 1 5A0D9E48
 P 4750 4450
-F 0 "C?" V 4600 4450 50  0000 L CNN
+F 0 "C5" V 4600 4450 50  0000 L CNN
 F 1 "300uF" H 4650 4250 50  0000 L CNN
-F 2 "" H 4788 4300 50  0001 C CNN
+F 2 "Capacitors_THT:CP_Radial_D8.0mm_P5.00mm" H 4788 4300 50  0001 C CNN
 F 3 "" H 4750 4450 50  0001 C CNN
 	1    4750 4450
@@
 Connection ~ 4900 4150
 Connection ~ 4600 4150
+Wire Wire Line
+	9750 1450 9750 1550
 $EndSCHEMATC
