File: esp8266-board/esp8266-board.sch (KiCad schematic (older format))
At the start: 25 parts, among them J1 PGM, J2 StepDown-3A, J3 LED, J4 USB, J5 Barrel_Jack, U1 ESP-12E, U2 AP2112, U3 AMS1117-3.3

Commit message: WIP
Parts:
- C1, C2, C3, C4: symbol C -> esp8266-board-rescue:C
- C5: symbol CP -> esp8266-board-rescue:CP
- J1: symbol Conn_01x05 -> esp8266-board-rescue:Conn_01x05
- J2: symbol StepDown-3A -> esp8266-board-rescue:StepDown-3A
- J3: symbol Conn_01x04 -> esp8266-board-rescue:Conn_01x04
- J4: symbol USB_OTG -> esp8266-board-rescue:USB_OTG
- J5: symbol Barrel_Jack -> esp8266-board-rescue:Barrel_Jack
- JP1, JP2, JP3: symbol Jumper_NO_Small -> esp8266-board-rescue:Jumper_NO_Small
- R1, R2, R3, R4, R5, R6, R7, R8: symbol R -> esp8266-board-rescue:R
- S1: symbol ROTARY_ENCODER_W_SPST -> esp8266-board-rescue:ROTARY_ENCODER_W_SPST
- U1: symbol ESP-12E -> esp8266-board-rescue:ESP-12E
- U2: symbol AP2112 -> esp8266-board-rescue:AP2112
- U3: symbol AMS1117-3.3 -> esp8266-board-rescue:AMS1117-3.3
Changed lines of the file:
@@
-EESchema Schematic File Version 2
-LIBS:power
-LIBS:device
-LIBS:transistors
-LIBS:conn
-LIBS:linear
-LIBS:regul
-LIBS:74xx
-LIBS:cmos4000
-LIBS:adc-dac
-LIBS:memory
-LIBS:xilinx
-LIBS:microcontrollers
-LIBS:dsp
-LIBS:microchip
-LIBS:analog_switches
-LIBS:motorola
-LIBS:texas
-LIBS:intel
-LIBS:audio
-LIBS:interface
-LIBS:digital-audio
-LIBS:philips
-LIBS:display
-LIBS:cypress
-LIBS:siliconi
-LIBS:opto
-LIBS:atmel
-LIBS:contrib
-LIBS:valves
-LIBS:switches_inputs
-LIBS:voltage-regulators
-LIBS:esp8266-board-cache
-EELAYER 25 0
+EESchema Schematic File Version 4
+EELAYER 30 0
 EELAYER END
 $Descr A4 11693 8268
@@
 $EndDescr
 $Comp
-L ESP-12E U1
+L esp8266-board-rescue:ESP-12E U1
 U 1 1 5A00CD38
 P 4800 2700
@@
 $EndComp
 $Comp
-L StepDown-3A J2
+L esp8266-board-rescue:StepDown-3A J2
 U 1 1 5A00ECE4
 P 8750 4400
@@
 $EndComp
 $Comp
-L USB_OTG J4
+L esp8266-board-rescue:USB_OTG J4
 U 1 1 5A00ED3B
 P 9850 2250
@@
 $EndComp
 $Comp
-L GND #PWR01
+L esp8266-board-rescue:GND #PWR01
 U 1 1 5A00ED9B
 P 9900 2850
@@
 	9850 2850 9900 2850
 $Comp
-L +5V #PWR02
+L esp8266-board-rescue:+5V #PWR02
 U 1 1 5A00EDDB
 P 10300 2050
@@
 	10150 2050 10300 2050
 $Comp
-L +5V #PWR03
+L esp8266-board-rescue:+5V #PWR03
 U 1 1 5A00EE6B
 P 8700 5300
@@
 $EndComp
 $Comp
-L GND #PWR04
+L esp8266-board-rescue:GND #PWR04
 U 1 1 5A00EE90
 P 8800 5100
@@
 	8700 4850 8700 5300
 $Comp
-L +3V3 #PWR05
+L esp8266-board-rescue:+3V3 #PWR05
 U 1 1 5A00EEDD
 P 9150 4900
@@
 $EndComp
 $Comp
-L Barrel_Jack J5
+L esp8266-board-rescue:Barrel_Jack J5
 U 1 1 5A00EF7E
 P 10050 1550
@@
 $EndComp
 $Comp
-L +5V #PWR06
+L esp8266-board-rescue:+5V #PWR06
 U 1 1 5A00EFBC
 P 9450 1650
@@
 	9450 1650 9750 1650
 $Comp
-L GND #PWR07
+L esp8266-board-rescue:GND #PWR07
 U 1 1 5A00EFE9
 P 9300 1450
@@
 	9300 1450 9750 1450
 $Comp
-L GND #PWR08
+L esp8266-board-rescue:GND #PWR08
 U 1 1 5A00F04B
 P 5900 3100
@@
 $EndComp
 $Comp
-L +3V3 #PWR09
+L esp8266-board-rescue:+3V3 #PWR09
 U 1 1 5A00F06B
 P 3250 3100
@@
 	3250 3100 3900 3100
 Wire Wire Line
-	5700 3100 6100 3100
-$Comp
-L +3V3 #PWR010
+	5700 3100 5900 3100
+$Comp
+L esp8266-board-rescue:+3V3 #PWR010
 U 1 1 5A00F0AA
 P 3450 2400
@@
 $EndComp
 $Comp
-L R R1
+L esp8266-board-rescue:R R1
 U 1 1 5A00F0E8
 P 3650 2400
@@
 	3500 2400 3450 2400
 Wire Wire Line
-	8800 4850 8800 5100
-Connection ~ 8800 5050
-Wire Wire Line
 	9150 4900 8900 4900
 Wire Wire Line
 	8900 4900 8900 4850
 $Comp
-L C C2
+L esp8266-board-rescue:C C2
 U 1 1 5A010134
 P 4750 4150
@@
 	3900 4150 3900 3100
 $Comp
-L +3V3 #PWR011
+L esp8266-board-rescue:+3V3 #PWR011
 U 1 1 5A01021B
 P 6500 2800
@@
 $EndComp
 $Comp
-L R R4
+L esp8266-board-rescue:R R4
 U 1 1 5A010263
 P 6350 2800
@@
 	5700 2800 6200 2800
 $Comp
-L R R5
+L esp8266-board-rescue:R R5
 U 1 1 5A0108BC
 P 6350 2900
@@
 	6200 2900 5700 2900
 $Comp
-L R R3
+L esp8266-board-rescue:R R3
 U 1 1 5A0109BD
 P 5950 3000
@@
 	5800 3000 5700 3000
 $Comp
-L R R2
+L esp8266-board-rescue:R R2
 U 1 1 5A010A6F
 P 3650 2600
@@
 GPIO13
 $Comp
-L Conn_01x05 J1
+L esp8266-board-rescue:Conn_01x05 J1
 U 1 1 5A0111F1
 P 6550 4900
@@
 $EndComp
 $Comp
-L GND #PWR012
+L esp8266-board-rescue:GND #PWR012
 U 1 1 5A01125D
 P 5850 4700
@@
 RX
 $Comp
-L Conn_01x04 J3
+L esp8266-board-rescue:Conn_01x04 J3
 U 1 1 5A011626
 P 3750 6700
@@
 $EndComp
 $Comp
-L GND #PWR013
+L esp8266-board-rescue:GND #PWR013
 U 1 1 5A0117FF
 P 3100 6700
@@
 	3100 6700 3550 6700
 Wire Wire Line
-	3150 6600 3550 6600
-$Comp
-L Jumper_NO_Small JP1
+	3150 6600 3350 6600
+$Comp
+L esp8266-board-rescue:Jumper_NO_Small JP1
 U 1 1 5A0119F3
 P 2350 3800
@@
 NoConn ~ 8600 4850
 $Comp
-L C C1
+L esp8266-board-rescue:C C1
 U 1 1 5A012B7F
 P 4750 3850
@@
 $EndComp
 Wire Wire Line
-	4900 3850 4900 4450
-Wire Wire Line
-	4600 3850 4600 4450
-$Comp
-L ROTARY_ENCODER_W_SPST S1
+	4900 3850 4900 4150
+Wire Wire Line
+	4600 3850 4600 4150
+$Comp
+L esp8266-board-rescue:ROTARY_ENCODER_W_SPST S1
 U 1 1 5A074E2B
 P 4200 5000
@@
 $EndComp
 $Comp
-L GND #PWR014
+L esp8266-board-rescue:GND #PWR014
 U 1 1 5A074EAE
 P 4200 5350
@@
 $EndComp
 Wire Wire Line
-	3750 5350 5000 5350
+	3750 5350 4200 5350
 Wire Wire Line
 	3750 5350 3750 5100
@@
 GPIO13
 $Comp
-L +3V3 #PWR015
+L esp8266-board-rescue:+3V3 #PWR015
 U 1 1 5A0763B7
 P 6700 4000
@@
 GPIO5
 $Comp
-L R R6
+L esp8266-board-rescue:R R6
 U 1 1 5A0768D9
 P 6500 4000
@@
 $EndComp
 $Comp
-L R R7
+L esp8266-board-rescue:R R7
 U 1 1 5A0768E1
 P 6500 4150
@@
 i2c resistors
 $Comp
-L Jumper_NO_Small JP3
+L esp8266-board-rescue:Jumper_NO_Small JP3
 U 1 1 5A0894A6
 P 3350 6500
@@
 $EndComp
 $Comp
-L Jumper_NO_Small JP2
+L esp8266-board-rescue:Jumper_NO_Small JP2
 U 1 1 5A08975F
 P 3150 6500
@@
 Connection ~ 3350 6600
 $Comp
-L +5V #PWR016
+L esp8266-board-rescue:+5V #PWR016
 U 1 1 5A08984D
 P 3350 6400
@@
 $EndComp
 $Comp
-L +3V3 #PWR017
+L esp8266-board-rescue:+3V3 #PWR017
 U 1 1 5A08989B
 P 3150 6400
@@
 Voltage Regulation\nPopulate only one
 $Comp
-L AMS1117-3.3 U3
+L esp8266-board-rescue:AMS1117-3.3 U3
 U 1 1 5A0C88E6
 P 9800 4250
@@
 $EndComp
 $Comp
-L +5V #PWR018
+L esp8266-board-rescue:+5V #PWR018
 U 1 1 5A0C895B
 P 9350 4250
@@
 $EndComp
 $Comp
-L +3V3 #PWR019
+L esp8266-board-rescue:+3V3 #PWR019
 U 1 1 5A0C89C1
 P 10300 4250
@@
 $EndComp
 $Comp
-L GND #PWR020
+L esp8266-board-rescue:GND #PWR020
 U 1 1 5A0C8A20
 P 9800 4700
@@
 	10100 4250 10300 4250
 $Comp
-L AP2112 U2
+L esp8266-board-rescue:AP2112 U2
 U 1 1 5A0C8E30
 P 9550 5850
@@
 $EndComp
 $Comp
-L +5V #PWR021
+L esp8266-board-rescue:+5V #PWR021
 U 1 1 5A0C8F35
 P 8800 5700
@@
 $EndComp
 $Comp
-L GND #PWR022
+L esp8266-board-rescue:GND #PWR022
 U 1 1 5A0C8F77
 P 9000 5850
@@
 	8800 5700 9100 5700
 $Comp
-L +3V3 #PWR023
+L esp8266-board-rescue:+3V3 #PWR023
 U 1 1 5A0C912A
 P 10250 5700
@@
 	10000 5700 10250 5700
 $Comp
-L R R8
+L esp8266-board-rescue:R R8
 U 1 1 5A0C9334
 P 8800 5850
@@
 Populate only one power jumper
 $Comp
-L C C3
+L esp8266-board-rescue:C C3
 U 1 1 5A087306
 P 9400 5000
@@
 $EndComp
 $Comp
-L +3V3 #PWR024
+L esp8266-board-rescue:+3V3 #PWR024
 U 1 1 5A0CC7AF
 P 9550 5000
@@
 $EndComp
 $Comp
-L GND #PWR025
+L esp8266-board-rescue:GND #PWR025
 U 1 1 5A0CC7F1
 P 9250 5000
@@
 $EndComp
 $Comp
-L +5V #PWR026
+L esp8266-board-rescue:+5V #PWR026
 U 1 1 5A0CCFB7
 P 9300 2050
@@
 $EndComp
 $Comp
-L GND #PWR027
+L esp8266-board-rescue:GND #PWR027
 U 1 1 5A0CCFF9
 P 9300 2350
@@
 $EndComp
 $Comp
-L C C4
+L esp8266-board-rescue:C C4
 U 1 1 5A0CD03B
 P 9300 2200
@@
 $EndComp
 $Comp
-L CP C5
+L esp8266-board-rescue:CP C5
 U 1 1 5A0D9E48
 P 4750 4450
@@
 Wire Wire Line
 	9750 1450 9750 1550
+Wire Wire Line
+	5900 3100 6100 3100
+Wire Wire Line
+	4200 5350 5000 5350
+Wire Wire Line
+	3350 6600 3550 6600
+Wire Wire Line
+	4900 4150 4900 4450
+Wire Wire Line
+	4600 4150 4600 4450
+Wire Wire Line
+	8800 4850 8800 5100
 $EndSCHEMATC
