File: esp8266-board/esp8266-board.kicad_pcb (KiCad board)
At the start: 2 copper layers, 59.4 x 59.4 mm, 26 parts, among them J1 PGM, J2 StepDown-3A, J3 LED, J4 USB, J5 Barrel_Jack, U1 ESP-12E, U2 AP2112, U3 AMS1117-3.3

Commit message: WIP
Parts:
- C5: value 300uF -> 220uF; footprint Capacitors_THT:CP_Radial_D8.0mm_P5.00mm -> Capacitors_Tantalum_SMD:CP_Tantalum_Case-B_EIA-3528-21_Hand
- J4: footprint Power:USB_Micro-B -> Connectors:USB_Micro-B
- moved C5 4.68 mm to (129.4, 107.4)
Connections:
- J2 pad 1: (no net) -> Net-(J2-Pad1)
- J4 pad 2: (no net) -> Net-(J4-Pad2)
- J4 pad 3: (no net) -> Net-(J4-Pad3)
- J4 pad 4: (no net) -> Net-(J4-Pad4)
- U1 pad 17: (no net) -> Net-(U1-Pad17)
- U1 pad 18: (no net) -> Net-(U1-Pad18)
- U1 pad 19: (no net) -> Net-(U1-Pad19)
- U1 pad 2: (no net) -> ADC
- U1 pad 20: (no net) -> Net-(U1-Pad20)
- U1 pad 21: (no net) -> Net-(U1-Pad21)
- U1 pad 22: (no net) -> Net-(U1-Pad22)
- U2 pad 4: (no net) -> Net-(U2-Pad4)
Routing:
- net GND: track 31.1 -> 34.1 mm, vias 6 -> 7
- net +3V3: track 105.4 -> 107.9 mm

Commit message: WIP
Connections:
- net ~FLASH renamed ~{FLASH}
- net ~RST renamed ~{RST}
Other:
- net class 3.3V PWR removed
- net class 5V PWR removed
- net class Default removed
