File: esp8266-pgm-adapter/esp8266-pgm-adapter.sch (KiCad schematic (older format))
At the start: 5 parts, among them J1 Conn_01x05, J2 Conn_01x03

Commit message: WIP
Parts:
- J1: symbol Conn_01x05 -> esp8266-pgm-adapter-rescue:Conn_01x05
- J2: symbol Conn_01x03 -> esp8266-pgm-adapter-rescue:Conn_01x03
- R1: symbol R -> esp8266-pgm-adapter-rescue:R
- S1, S2: symbol TAC_SWITCH_6x6mm -> esp8266-pgm-adapter-rescue:TAC_SWITCH_6x6mm
Changed lines of the file:
@@
-EESchema Schematic File Version 2
-LIBS:power
-LIBS:device
-LIBS:switches
-LIBS:relays
-LIBS:motors
-LIBS:transistors
-LIBS:conn
-LIBS:linear
-LIBS:regul
-LIBS:74xx
-LIBS:cmos4000
-LIBS:adc-dac
-LIBS:memory
-LIBS:xilinx
-LIBS:microcontrollers
-LIBS:dsp
-LIBS:microchip
-LIBS:analog_switches
-LIBS:motorola
-LIBS:texas
-LIBS:intel
-LIBS:audio
-LIBS:interface
-LIBS:digital-audio
-LIBS:philips
-LIBS:display
-LIBS:cypress
-LIBS:siliconi
-LIBS:opto
-LIBS:atmel
-LIBS:contrib
-LIBS:valves
-LIBS:switches_inputs
+EESchema Schematic File Version 4
 LIBS:esp8266-pgm-adapter-cache
-EELAYER 25 0
+EELAYER 26 0
 EELAYER END
 $Descr A4 11693 8268
@@
 $EndDescr
 $Comp
-L Conn_01x05 J1
+L esp8266-pgm-adapter-rescue:Conn_01x05 J1
 U 1 1 5A2DC871
 P 3400 2800
@@
 ~FLASH
 $Comp
-L TAC_SWITCH_6x6mm S1
+L esp8266-pgm-adapter-rescue:TAC_SWITCH_6x6mm S1
 U 1 1 5A2DC905
 P 4700 2800
@@
 ~FLASH
 $Comp
-L R R1
+L esp8266-pgm-adapter-rescue:R R1
 U 1 1 5A2DC95F
 P 4250 2750
@@
 GND
 $Comp
-L TAC_SWITCH_6x6mm S2
+L esp8266-pgm-adapter-rescue:TAC_SWITCH_6x6mm S2
 U 1 1 5A2DCB56
 P 4700 3600
@@
 GND
 $Comp
-L Conn_01x03 J2
+L esp8266-pgm-adapter-rescue:Conn_01x03 J2
 U 1 1 5A2DCBD5
 P 5750 2600
