File: esp8266-pgm-adapter/esp8266-pgm-adapter.kicad_pcb (KiCad board)
At the start: 2 copper layers, 27 x 15 mm, 5 parts, among them J1 Conn_01x05, J2 Conn_01x03

Commit message: WIP
Connections:
- net /~FLASH renamed /~{FLASH}
- net /~RST renamed /~{RST}
Other:
- net class Default removed
